Commit message: Correction in a sample urdf.

File: test/sample_smurfs/two_boxes_joined/urdf/two_boxes.urdf (robot description, URDF)
Before this commit: robot spaceclimber, 2 links, 1 joints
Links:
- removed link box2
- added link box, mass 1.121; collision box size=0.1 0.1 0.1; visual box size=0.1 0.1 0.1
Joints:
- removed joint rootbox2
- added joint root2box: type fixed, parent root, child box, origin xyz=0.41 0. 0. rpy=0 0 0, axis 0.0 1.0 0, limit lower=-0.785398 upper=0.785398 effort=1000 velocity=6.28

Commit message: Normally the joints and the motor are named like the target of the transformations

File: test/sample_smurfs/two_boxes_joined/urdf/two_boxes.urdf (robot description, URDF)
Before this commit: robot spaceclimber, 2 links, 1 joints
Joints:
- removed joint root2box
- added joint box: type fixed, parent root, child box, origin xyz=0.41 0. 0. rpy=0 0 0, axis 0.0 1.0 0, limit lower=-0.785398 upper=0.785398 effort=1000 velocity=6.28

File: test/sample_smurfs/two_boxes_joined/urdf/two_boxes_dynamic_joint.urdf (robot description, URDF)
Before this commit: robot spaceclimber, 2 links, 1 joints
Joints:
- removed joint root2box
- added joint box: type revolute, parent root, child box, origin xyz=0.41 0. 0. rpy=0 0 0, axis 0.0 1.0 0, limit lower=-0.785398 upper=0.785398 effort=1000 velocity=6.28
