Commit message: Now The example of the two boxes is more useful for testing

File: test/sample_smurfs/two_boxes_joined/urdf/two_boxes_dynamic_joint.urdf (robot description, URDF)
Before this commit: robot spaceclimber, 2 links, 1 joints
Links:
- added link box2, mass 1.121; collision box size=0.1 0.1 0.1; visual box size=0.1 0.1 0.1
- link root: geometry collision box size=0.2 0.2 2.2; visual box size=0.2 0.2 2.2
Joints:
- added joint box2: type revolute, parent box, child box2, origin xyz=0.41 0. 0. rpy=0 0 0, axis 0.0 1.0 0.0, limit lower=-0.785398 upper=0.785398 effort=1000 velocity=6.28
- joint box: axis 0.0 1.0 0 -> 0.0 1.0 0.0; origin xyz=0.41 0. 0. rpy=0 0 0 -> xyz=0. 0. 0. rpy=0 0 0; type revolute -> fixed
